File: Power.kicad_sch (KiCad schematic)
At the start: 18 parts, among them J4 PJ-102AH, Q1 PMV48XP, U1 NCP1117-5.0_SOT223, U6 LP2985-3.3, U7 LMV358IDGKR

Commit message: WIP, replace bottom headers
replaced the two bottom headers with one big 2x16 header.
Changed lines of the file:
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@@
 (kicad_sch
-	(version 20231120)
+	(version 20250114)
 	(generator "eeschema")
-	(generator_version "8.0")
+	(generator_version "9.0")
 	(paper "A4")
 	(title_block
