File: Arduino Mega 2560.kicad_pcb (KiCad board)
At the start: 2 copper layers, 68.6 x 53.3 mm, 62 parts, among them J1 USB_C_Receptacle_USB2.0_16P, J11 PPTC081LFBN-RC, J12 M20-9980345, J13 Conn_01x20, J2 M20-9980345, J3 M20-9980245, J4 PJ-102AH, J5 PPTC182LFBN-RC, J9 PPTC082LFBN-RC, Q1 PMV48XP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

Commit message: Continued routing
All pins except 3.3v are hooked up. Rerouted lots of traces to no longer produce vias in silkscreen area
Routing:
- net RESET: track 11.9 -> 109.0 mm, vias 2 -> 6
- net Net-(D6-A): track 0.00 -> 67.6 mm, vias 0 -> 2
- net GND: track 151.4 -> 217.1 mm, vias 11 -> 12
- net XTAL2: track 3.31 -> 34.8 mm, vias 0 -> 6
- net XTAL1: track 3.31 -> 32.3 mm, vias 0 -> 4
- net PB7: track 62.6 -> 90.7 mm, vias 1 -> 4
- net PC4: track 50.7 -> 27.6 mm, vias 1 -> 0
- net PC5: track 46.2 -> 24.5 mm, vias 1 -> 0
- net PG2: track 53.0 -> 31.8 mm, vias 1 -> 0
- net AREF: track 59.0 -> 76.0 mm, vias 1 -> 2
- net PC6: track 48.0 -> 32.2 mm, vias 1 -> 0
- net SCL: track 89.8 -> 101.1 mm
- net +5V: track 155.8 -> 145.2 mm, vias 5 -> 6
- net RESET2: track 0.00 -> 9.04 mm
- net PL0: track 37.0 -> 43.8 mm
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Other:
- board text added: "11~ 10~"
- board text added: "13 12"
- board text added: "3~"
- board text added: "5~"
- board text added: "6~"
- board text added: "9~ 8 7"
- board text added: "SCL SDA GND"
- board text added: "↑"
- board text removed: "13"

Commit message: WIP, replace bottom headers
replaced the two bottom headers with one big 2x16 header.
Parts:
- removed J9: PPTC082LFBN-RC, Connector_PinSocket_2.54mm:PinSocket_2x08_P2.54mm_Vertical
- added J6: Conn_02x16_Top_Bottom, Connector_PinSocket_2.54mm:PinSocket_2x16_P2.54mm_Vertical, F.Cu at (160.6, 129.5)
- added JP1: SolderJumper_2_Open, Jumper:SolderJumper-2_P1.3mm_Open_Pad1.0x1.5mm, F.Cu at (191.0, 97.4)
- moved FID4 93.3 mm to (191.1, 93.3)
- moved C4 8.25 mm to (105.7, 108.8), turned to 0 degrees
- moved C14 8.11 mm to (111.2, 113.7), turned to -90 degrees
- moved RN5 7.19 mm to (109.0, 114.0)
- moved D4 7.12 mm to (114.7, 122.5)
- moved C1 6.78 mm to (115.8, 115.8)
- moved C2 6.77 mm to (123.0, 115.8)
- moved D7 5.56 mm to (130.0, 112.9)
- moved C9 5.40 mm to (115.8, 109.2)
- moved C3 5.34 mm to (128.0, 113.5)
- moved J11 5.26 mm to (140.0, 134.8)
- moved Y1 5.23 mm to (132.5, 116.2)
- moved U7 5.14 mm to (111.0, 110.2)
- moved RN4 4.98 mm to (132.6, 112.5)
- moved R1 4.53 mm to (134.5, 116.1)
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Routing:
- net GND: track 217.1 -> 149.3 mm, vias 12 -> 8
- net VCC: track 50.5 -> 0.00 mm, vias 3 -> 0
- net +5V: track 145.2 -> 103.7 mm
- net RESET: track 109.0 -> 92.5 mm, vias 6 -> 3
- net XTAL1: track 32.3 -> 22.0 mm
- net XTAL2: track 34.8 -> 25.1 mm
- net PE0: track 66.2 -> 56.9 mm
- net CMP: track 9.15 -> 0.00 mm
- net PE1: track 66.6 -> 57.6 mm
- net Net-(D4-A): track 8.28 -> 0.00 mm
- net GATE_CMD: track 8.25 -> 1.37 mm, vias 2 -> 0
- net PB7: track 90.7 -> 89.3 mm, vias 4 -> 3
- net ADC7: track 25.6 -> 26.8 mm
- net ADC15: track 25.3 -> 24.3 mm
- net L13: track 0.65 -> 0.00 mm
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
Commit message: Continued work
almost complete
Parts:
- removed J11: PPTC081LFBN-RC, Connector_PinSocket_2.54mm:PinSocket_1x08_P2.54mm_Vertical
- JP1: moved to B.Cu
- moved FID4 83.4 mm to (114.5, 126.5)
- moved JP1 75.7 mm to (118.3, 118.8)
- moved C6 16.9 mm to (117.5, 129.5), turned to 180 degrees
- moved C12 5.37 mm to (124.0, 105.2)
- moved C5 5.00 mm to (128.8, 102.8), turned to 90 degrees
- moved D1 4.59 mm to (129.3, 105.5)
- moved D2 4.08 mm to (129.3, 107.5)
- moved RN3 3.21 mm to (126.0, 102.7), turned to 90 degrees
- moved C14 3.19 mm to (110.2, 116.8), turned to 0 degrees
- moved JP2 2.35 mm to (121.3, 109.8)
- moved C9 1.58 mm to (117.2, 109.8)
- moved RN5 1.50 mm to (110.5, 114.0)
- moved C7 1.03 mm to (142.3, 119.8)
- moved J6 0.95 mm to (159.7, 129.5)
- moved RV1 0.84 mm to (107.8, 99.0), turned to 180 degrees
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Connections:
- J6 pad 17: unconnected-(J6-Pin_17-Pad17) -> VCC
- J6 pad 18: unconnected-(J6-Pin_18-Pad18) -> VCC
- J6 pad 19: unconnected-(J6-Pin_19-Pad19) -> GND
- J6 pad 20: unconnected-(J6-Pin_20-Pad20) -> GND
- J6 pad 21: unconnected-(J6-Pin_21-Pad21) -> GND
- J6 pad 22: unconnected-(J6-Pin_22-Pad22) -> GND
- J6 pad 23: unconnected-(J6-Pin_23-Pad23) -> GND
- J6 pad 24: unconnected-(J6-Pin_24-Pad24) -> GND
- J6 pad 25: unconnected-(J6-Pin_25-Pad25) -> +3.3V
- J6 pad 26: unconnected-(J6-Pin_26-Pad26) -> +3.3V
- J6 pad 27: unconnected-(J6-Pin_27-Pad27) -> +5V
- J6 pad 28: unconnected-(J6-Pin_28-Pad28) -> +5V
- J6 pad 29: unconnected-(J6-Pin_29-Pad29) -> +5V
- J6 pad 30: unconnected-(J6-Pin_30-Pad30) -> +5V
- J6 pad 31: unconnected-(J6-Pin_31-Pad31) -> +5V
- J6 pad 32: unconnected-(J6-Pin_32-Pad32) -> RESET
Routing:
- net +5V: track 103.7 -> 308.4 mm, vias 6 -> 14
- net GND: track 149.3 -> 286.3 mm, vias 8 -> 171
- net RESET: track 92.5 -> 185.9 mm, vias 3 -> 9
- net RESET2: track 9.04 -> 83.6 mm, vias 0 -> 4
- net VCC: track 0.00 -> 69.8 mm, vias 0 -> 2
- net +3.3V: track 0.00 -> 43.6 mm, vias 0 -> 3
- net DTR: track 0.00 -> 35.4 mm, vias 0 -> 2
- net M8TXD: track 0.00 -> 25.8 mm, vias 0 -> 2
- net L13: track 0.00 -> 25.2 mm, vias 0 -> 2
- net M8RXD: track 0.00 -> 24.4 mm, vias 0 -> 2
- net RXL: track 0.00 -> 23.0 mm, vias 0 -> 2
- net TXL: track 0.00 -> 20.8 mm, vias 0 -> 2
- net D-: track 0.00 -> 20.0 mm, vias 0 -> 2
- net Net-(U4-UCAP): track 0.00 -> 19.7 mm, vias 0 -> 2
- net D+: track 0.00 -> 15.9 mm, vias 0 -> 2
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Other:
- board text added: "A0"
- board text added: "A1"
- board text added: "A10"
- board text added: "A11"
- board text added: "A12"
- board text added: "A13"
- board text added: "A14"
- board text added: "A15"
- board text added: "A16"
- board text added: "A2"
- board text added: "A3"
- board text added: "A5"
- board text added: "A6"
- board text added: "A7"
- board text added: "A8"
- board text added: "A9"
- board text removed: "10"
- board text removed: "11"
- board text removed: "12"
- board text removed: "3"
- board text removed: "5"
- board text removed: "6"
- board text removed: "7"
- board text removed: "8"
- board text removed: "9"
- board text removed: "A0 A1 A2 A3 A4 A5 A6 A7"
- board text removed: "A8 A9 A10 A11 A12 A13 A14 A15"
